File: VibHub32_1.0/2.1/vh_21c.sch (EAGLE design)
At the start: 97 parts, among them Q1 MOSFET_PCH-DMG2305UX-13, Q3 2N7002, U1 DRV8833C, U2 DRV8833C, U3 3.3V, U4 MAX16054AZT+T, U5 CH340C, U6 ESP-WROOM32

Commit message: Unsaved changes from last commit
Parts:
- R33: value 100K -> >1M
Changed lines of the file:
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@@
 <part name="Q3" library="vibhud" library_urn="urn:adsk.eagle:library:2530795" deviceset="MOSFET-NCH" device="-BSS138" package3d_urn="urn:adsk.eagle:package:2531077/3" value="2N7002"/>
 <part name="SUPPLY22" library="vibhud" library_urn="urn:adsk.eagle:library:2530795" deviceset="V_USB" device=""/>
-<part name="R33" library="vibhud" library_urn="urn:adsk.eagle:library:2530795" deviceset="RESISTOR" device="0805" package3d_urn="urn:adsk.eagle:package:2531030/3" value="100K"/>
+<part name="R33" library="vibhud" library_urn="urn:adsk.eagle:library:2530795" deviceset="RESISTOR" device="0805" package3d_urn="urn:adsk.eagle:package:2531030/3" value="&gt;1M"/>
 <part name="R35" library="vibhud" library_urn="urn:adsk.eagle:library:2530795" deviceset="RESISTOR" device="0805" package3d_urn="urn:adsk.eagle:package:2531030/3" value="150"/>
 <part name="GND31" library="vibhud" library_urn="urn:adsk.eagle:library:2530795" deviceset="GND" device=""/>
